Commit message: fixed xacro file to open in gazebo

File: rover_description/UVicArm.xacro (robot description, xacro)
@@ -38,9 +38,11 @@
   <xacro:property name="gripper_xyz" value="6 -34.8 80" />
   <link name="base_link">
-    <visual>
+    <xacro:default_inertial mass="1.8"/>
+    <visual name="">
       <geometry>
         <mesh filename="${filepath}BaseMotor.STL"/>
       </geometry>
       <origin rpy="${base_link_rpy}" xyz="${base_link_xyz}"/>
+      <material name=""/>
     </visual>
     <collision>

Commit message: Fix issues with Gazebo crashing

File: rover_description/UVicArm.xacro (robot description, xacro)
@@ -22,5 +22,5 @@
       <origin xyz="0 0 0" rpy="0 0 0"/>
       <mass value="${mass}" />
-      <inertia ixx="0.001" ixy="0.0" ixz="0.0" iyy="0.001" iyz="0.0" izz="0.001"/>
+      <inertia ixx="100" ixy="0.0" ixz="0.0" iyy="100" iyz="0.0" izz="100"/>
     </inertial>
   </xacro:macro>
@@ -37,6 +37,10 @@
   <xacro:property name="gripper_rpy" value="0 3.14 0" />
   <xacro:property name="gripper_xyz" value="6 -34.8 80" />
+  <link name="world"/>
+  <joint name="fixed" type="fixed">
+    <parent link="world"/>
+    <child link="base_link"/>
+  </joint>
   <link name="base_link">
-    <xacro:default_inertial mass="1.8"/>
     <visual name="">
       <geometry>
@@ -52,4 +56,5 @@
       <origin rpy="${base_link_rpy}" xyz="${base_link_xyz}"/>
     </collision>
+    <xacro:default_inertial mass="1000"/>
   </link>
   <link name="base_component">
@@ -67,5 +72,5 @@
       <origin rpy="${base_component_rpy}" xyz="${base_component_xyz}"/>
     </collision>
-    <xacro:default_inertial mass="1.8"/>
+    <xacro:default_inertial mass="1000"/>
   </link>
   <link name="shoulder">
@@ -83,5 +88,5 @@
       <origin rpy="${shoulder_rpy}" xyz="${shoulder_xyz}"/>
     </collision>
-    <xacro:default_inertial mass="1.1"/>
+    <xacro:default_inertial mass="1000"/>
   </link>
   <link name="elbow_link">
@@ -99,5 +104,5 @@
       <origin rpy="${elbow_link_rpy}" xyz="${elbow_link_xyz}"/>
     </collision>
-    <xacro:default_inertial mass="1.1"/>
+    <xacro:default_inertial mass="1000"/>
   </link>
   <link name="wrist_link">
@@ -115,5 +120,5 @@
       <origin rpy="${wrist_link_rpy}" xyz="${wrist_link_xyz}"/>
     </collision>
-    <xacro:default_inertial mass="0.382"/>
+    <xacro:default_inertial mass="1000"/>
   </link>
   <link name="gripper">
@@ -131,5 +136,5 @@
       <origin rpy="${gripper_rpy}" xyz="${gripper_xyz}"/>
     </collision>
-    <xacro:default_inertial mass="0.250"/>
+    <xacro:default_inertial mass="100"/>
   </link>
   <joint name="base_motor_to_base" type="continuous">
