Commit message: added collision tag to urdf file

File: rover_description/UVicArm.urdf (robot description, URDF)
Before this commit: robot UVicArm, 6 links, 5 joints
Links:
- link base_component: geometry collision mesh filename=package://uvic_rover/rover_description/Arm/BaseComponent.STL; visual mesh filename=package://uvic_rover/rover_description/Arm/BaseComponent.STL
- link base_link: geometry collision mesh filename=package://uvic_rover/rover_description/Arm/BaseMotor.STL; visual mesh filename=package://uvic_rover/rover_description/Arm/BaseMotor.STL
- link elbow_link: geometry collision mesh filename=package://uvic_rover/rover_description/Arm/ElbowLink2.STL; visual mesh filename=package://uvic_rover/rover_description/Arm/ElbowLink2.STL
- link gripper: geometry collision mesh filename=package://uvic_rover/rover_description/Arm/Gripper.STL; visual mesh filename=package://uvic_rover/rover_description/Arm/Gripper.STL
- link shoulder: geometry collision mesh filename=package://uvic_rover/rover_description/Arm/Shoulder.STL; visual mesh filename=package://uvic_rover/rover_description/Arm/Shoulder.STL
- link wrist_link: geometry collision mesh filename=package://uvic_rover/rover_description/Arm/Wrist.STL; visual mesh filename=package://uvic_rover/rover_description/Arm/Wrist.STL

Commit message: Adding dummy interial tags

File: rover_description/UVicArm.urdf (robot description, URDF)
Before this commit: robot UVicArm, 6 links, 5 joints
Links:
- link base_component: mass None -> 1.8
- link elbow_link: mass None -> 1.1
- link gripper: mass None -> 0.250
- link shoulder: mass None -> 1.1
- link wrist_link: mass None -> 0.382

Commit message: added group name for moveit

File: rover_description/UVicArm.urdf (robot description, URDF)
Before this commit: robot UVicArm, 6 links, 5 joints
Joints:
- removed joint base_motor_to_base
- removed joint base_to_shoulder
- removed joint elbow_to_wrist
- removed joint shoulder_to_elbow
- removed joint wrist_to_gripper
